File: GameSystems/SG/GG/Cartridge/Cartridge.kicad_pcb (KiCad board)
At the start: 2 copper layers, 60.1 x 63.1 mm, 1 part, among them J1 SG_GG_CARTRIDGE_FINGERS

Commit message: Reorganizing
- Moved symbol and footprint libraries to a dedicated library folder.
- Renamed symbol and foot print libraries to names based on the manufacturer of the targeted devices.
- Clarified symbol, footprint, and library descriptions.
- Updated and added READMEs.
- Added images for symbols, footprints, and PCBs.
- Added trademark disclaimers.
Parts:
- J1: footprint !GGFootprints:SG_GG_CARTRIDGE_FINGERS -> !SGFootprints:SG_GG_CARTRIDGE_FINGERS
Changed lines of the file:
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@@
   (net 38 "unconnected-(J1-Pad44)")
   (net 39 "unconnected-(J1-Pad45)")
-  (footprint "!GGFootprints:SG_GG_CARTRIDGE_FINGERS" (layer "F.Cu")
+  (footprint "!SGFootprints:SG_GG_CARTRIDGE_FINGERS" (layer "F.Cu")
     (at 150 103.34)
-    (descr "GG cartridge fingers (for cart PCBs)")
+    (descr "Game Gear-compatible cartridge fingers (for replacement PCBs, flash cartridges, etc.)")
+    (tags "Sega, Game Gear, cartridge fingers")
     (property "Copyright" "©2022 StarshadeRETRO")
+    (property "Disclaimer" "SEGA and Game Gear are registered trademarks of SEGA GAMES CO., LTD. Not sponsored, endorsed, or approved by SEGA.")
     (property "License" "BSD-3-Clause")
     (property "Sheetfile" "Cartridge.kicad_sch")
@@
       (effects (font (size 1 1) (thickness 0.15)))
     )
-    (fp_text user "CARD EDGE" (at 30.595 2.144 90 unlocked) (layer "Cmts.User")
-      (effects (font (size 0.5 0.5) (thickness 0.1)))
-    )
-    (fp_text user "©2022 StarshadeRETRO; License: BSD-3-Clause" (at 0 6.9) (layer "Cmts.User")
+    (fp_text user "CARD EDGE" (at -30.65 2.444 270 unlocked) (layer "Cmts.User")
       (effects (font (size 0.5 0.5) (thickness 0.1)))
     )
@@
       (effects (font (size 0.5 0.5) (thickness 0.1)))
     )
-    (fp_text user "CARD EDGE" (at -30.65 2.444 270 unlocked) (layer "Cmts.User")
+    (fp_text user "SEGA and Game Gear are registered trademarks of SEGA GAMES CO., LTD. Not sponsored, endorsed, or approved by SEGA." (at 0 8) (layer "Cmts.User")
+      (effects (font (size 0.4 0.4) (thickness 0.08)))
+    )
+    (fp_text user "©2022 StarshadeRETRO; License: BSD-3-Clause" (at 0 6.9) (layer "Cmts.User")
+      (effects (font (size 0.5 0.5) (thickness 0.08)))
+    )
+    (fp_text user "CARD EDGE" (at 30.595 2.144 90 unlocked) (layer "Cmts.User")
       (effects (font (size 0.5 0.5) (thickness 0.1)))
     )
@@
     (fp_line (start -30.03 -6.436) (end -30.03 4.614) (layer "Dwgs.User") (width 0.12))
     (fp_line (start -30.03 4.614) (end 29.97 4.614) (layer "Dwgs.User") (width 0.12))
-    (fp_line (start 30.23 4.444) (end 30.34 4.524) (layer "Cmts.User") (width 0.12))
+    (fp_line (start 30.23 4.444) (end 30.34 4.364) (layer "Cmts.User") (width 0.12))
     (fp_line (start -30.285 0.144) (end -30.395 0.064) (layer "Cmts.User") (width 0.12))
-    (fp_line (start -30.285 0.144) (end -30.395 0.224) (layer "Cmts.User") (width 0.12))
+    (fp_line (start -29.93 4.804) (end -30.01 4.914) (layer "Cmts.User") (width 0.12))
     (fp_line (start -29.93 5.454) (end -29.93 4.804) (layer "Cmts.User") (width 0.12))
-    (fp_line (start -29.93 4.804) (end -30.01 4.914) (layer "Cmts.User") (width 0.12))
-    (fp_line (start -30.935 0.144) (end -30.285 0.144) (layer "Cmts.User") (width 0.12))
-    (fp_line (start 30.23 4.444) (end 30.34 4.364) (layer "Cmts.User") (width 0.12))
     (fp_line (start 30.88 4.444) (end 30.23 4.444) (layer "Cmts.User") (width 0.12))
     (fp_line (start -29.93 4.804) (end -29.85 4.914) (layer "Cmts.User") (width 0.12))
+    (fp_line (start -30.285 0.144) (end -30.395 0.224) (layer "Cmts.User") (width 0.12))
+    (fp_line (start -30.935 0.144) (end -30.285 0.144) (layer "Cmts.User") (width 0.12))
+    (fp_line (start 30.23 4.444) (end 30.34 4.524) (layer "Cmts.User") (width 0.12))
     (fp_rect (start -30.03 4.614) (end 29.97 -6.426) (layer "F.CrtYd") (width 0.12) (fill none))
+    (fp_line (start -7.65 4.878) (end -7.73 4.988) (layer "F.Fab") (width 0.12))
+    (fp_line (start 22.83 5.599) (end 22.83 4.949) (layer "F.Fab") (width 0.12))
     (fp_line (start 22.83 4.949) (end 22.91 5.059) (layer "F.Fab") (width 0.12))
-    (fp_line (start -7.65 5.528) (end -7.65 4.878) (layer "F.Fab") (width 0.12))
     (fp_line (start 22.83 4.949) (end 22.75 5.059) (layer "F.Fab") (width 0.12))
     (fp_line (start -7.65 4.878) (end -7.57 4.988) (layer "F.Fab") (width 0.12))
-    (fp_line (start -7.65 4.878) (end -7.73 4.988) (layer "F.Fab") (width 0.12))
-    (fp_line (start 22.83 5.599) (end 22.83 4.949) (layer "F.Fab") (width 0.12))
+    (fp_line (start -7.65 5.528) (end -7.65 4.878) (layer "F.Fab") (width 0.12))
     (pad "1" connect roundrect (at -27.97 2.48) (size 1.82 4) (layers "F.Cu" "F.Mask") (roundrect_rratio 0.25)
       (chamfer_ratio 0) (chamfer bottom_left bottom_right)
@@
       (chamfer_ratio 0) (chamfer bottom_left bottom_right)
       (net 39 "unconnected-(J1-Pad45)") (pinfunction "TV_Audio_L") (pintype "input+no_connect") (zone_connect 2))
-    (group "" (id 2e2e4a94-725e-4f49-b404-f43ade85681b)
-      (members
-        325609bf-7847-4d67-9403-f4c31541e5ce
-        4fc597e7-8428-4f51-b498-923939aa5782
-        b04e28cc-286f-4a9b-8132-5fe5394cd7cf
-      )
-    )
-    (group "" (id 342fcf22-9b1d-4514-ba5d-ce3f24feb242)
-      (members
-        61fb0432-baf6-4ed0-8468-5296f6162173
-        710ca3c3-3ad1-4f5d-b964-bb0981030c6c
-      )
-    )
-    (group "" (id 710ca3c3-3ad1-4f5d-b964-bb0981030c6c)
-      (members
-        2f8ca4e7-2188-44b5-b187-817a6d952437
-        bac19a77-e745-4550-ab80-25fa47b6cc5e
-        cc31d48f-68ba-4246-85ae-3915b1b333ed
-      )
-    )
-    (group "" (id 97d00f81-d9a8-4463-8b9f-9df13b90db94)
-      (members
-        95bce22d-f1db-4d7e-a03c-687daa86aaf3
-        d44edbd3-0a9f-4ee9-ae36-d3fe8e02b096
-      )
-    )
-    (group "" (id ae5eeb47-87d4-4264-b170-589036441130)
-      (members
-        0fc31e1c-da2b-4680-a236-1b46ee0826f1
-        429a5aa1-345d-4557-b061-7e1e26e17e8d
-        fc7cea58-cfd0-49e9-87cf-6275067fa432
-      )
-    )
-    (group "" (id c76fd29e-1e43-4ebf-86b9-b4c3b8d4d3c0)
-      (members
-        3d567e0a-ceef-4e72-86b3-7fa1f2019fb6
-        b6487df3-2db6-471a-9c44-177b196f1aac
-        e87a8ea0-bfd6-4c88-ba6d-22a200ace202
-      )
-    )
-    (group "" (id d44edbd3-0a9f-4ee9-ae36-d3fe8e02b096)
-      (members
-        82c4ff26-3314-450a-9ee5-d5238a79731d
-        a85e1b6f-455e-4c97-86fa-f33cf1acbe21
-        cf143a8c-dd6a-4de3-80e0-641957422496
-      )
-    )
-    (group "" (id dd877322-0c32-40ab-8651-c72a5281c63f)
-      (members
-        2e2e4a94-725e-4f49-b404-f43ade85681b
-        f8888daa-7449-4628-9a0f-c4c7a76da442
-      )
-    )
+    (group "" (id 3edde107-29e5-47b8-b333-9f2169675ae2)
+      (members
+        45ebbad4-4dac-47a1-bc38-ecbf507966fa
+        c66c7b25-56df-4612-8511-a7f8c68f9f62
+      )
+    )
+    (group "" (id 4cde4c73-a172-4faf-959e-9283e1c31aaa)
+      (members
+        f17bd064-0106-48d8-b841-6531b497b720
+        fa3f99f7-c626-4b84-b0dd-7a8c4f54ccab
+      )
+    )
+    (group "" (id 66358a56-beff-4fb1-8c3b-f3a345ef4c99)
+      (members
+        2c666f59-9e04-4d29-a8d4-868461f2da52
+        834768ce-e2ca-42c3-8c06-dc4d47c9c886
+      )
+    )
+    (group "" (id 693acd9b-f013-48db-88c8-8d5ad4842a4b)
+      (members
+        653bd0ac-a379-4bd9-8291-38dbb5cdef91
+        654f4e16-0d54-4ddf-bf06-6aaf05f300ce
+        745dc158-258e-4725-a839-23767e1177df
+      )
+    )
+    (group "" (id 7f345282-0af7-4297-b662-391e371123d5)
+      (members
+        064d3f04-8b49-49ef-8a20-3c44dfba7ae0
+        8d49d213-d837-4760-8f08-0ef01ebcd682
+        df7343e7-4f4d-4a9d-b9a9-0cc32fca2798
+      )
+    )
+    (group "" (id 834768ce-e2ca-42c3-8c06-dc4d47c9c886)
+      (members
+        30b57dde-8dbb-483f-88d7-c20cddf69b7d
+        a1278d7f-e034-41c1-825f-6817d2b27bda
+        ada88bef-ba19-470a-a67b-c0805db35fbe
+      )
+    )
+    (group "" (id c66c7b25-56df-4612-8511-a7f8c68f9f62)
+      (members
+        44bbb8b2-e684-4e77-8d4d-f4fe367668db
+        4e9aa5e0-67bb-4d00-87da-e303e2382671
+        9386b855-b057-4c09-a7ec-fef95f1cb1a5
+      )
+    )
+    (group "" (id f17bd064-0106-48d8-b841-6531b497b720)
+      (members
+        0f49b6a2-655f-465d-919b-44a41eb1d089
+        7036f495-346c-45db-8269-8b751ee1c847
+        ea4305ab-122e-4c51-b835-53f420ed8fcf
+      )
+    )
