File: GameSystems/SG/GG/Cartridge/Cartridge.kicad_sch (KiCad schematic)
At the start: 1 part, among them J1 SG_GG_CARTRIDGE_FINGERS

Commit message: Reorganizing
- Moved symbol and footprint libraries to a dedicated library folder.
- Renamed symbol and foot print libraries to names based on the manufacturer of the targeted devices.
- Clarified symbol, footprint, and library descriptions.
- Updated and added READMEs.
- Added images for symbols, footprints, and PCBs.
- Added trademark disclaimers.
Parts:
- J1: footprint !GGFootprints:SG_GG_CARTRIDGE_FINGERS -> !SGFootprints:SG_GG_CARTRIDGE_FINGERS; symbol !GGSymbols:SG_GG_CARTRIDGE_FINGERS -> !SGSymbols:SG_GG_CARTRIDGE_FINGERS; Disclaimer (none) -> SEGA and Game Gear are registered trademarks of SEGA GAMES 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
Other:
- company: (none) -> ©2022 StarshadeRETRO; License: BSD-3-Clause
- title: (none) -> Game Gear-compatible Cartridge Template
Changed lines of the file:
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@@
 (kicad_sch (version 20211123) (generator eeschema)
   (paper "A4")
+  (title_block
+    (title "Game Gear-compatible Cartridge Template")
+    (date "2022-12-15")
+    (rev "1")
+    (company "©2022 StarshadeRETRO; License: BSD-3-Clause")
+    (comment 1 "Not sponsored, endorsed, or approved by SEGA.")
+    (comment 2 "SEGA and Game Gear are registered trademarks of SEGA GAMES CO., LTD.")
+  )
   (junction (at 170.18 82.55) (diameter 0) (color 0 0 0 0)
   )
@@
     (pin "1")
   )
-  (symbol (lib_id "!GGSymbols:SG_GG_CARTRIDGE_FINGERS") (at 142.24 88.9 0) (unit 1)
+  (symbol (lib_id "!SGSymbols:SG_GG_CARTRIDGE_FINGERS") (at 142.24 88.9 0) (unit 1)
     (in_bom no) (on_board yes) (fields_autoplaced)
     (property "Reference" "J1" (id 0) (at 142.24 54.61 0))
     (property "Value" "SG_GG_CARTRIDGE_FINGERS" (id 1) (at 142.24 57.15 0))
-    (property "Footprint" "!GGFootprints:SG_GG_CARTRIDGE_FINGERS" (id 2) (at 142.24 54.61 0)
+    (property "Footprint" "!SGFootprints:SG_GG_CARTRIDGE_FINGERS" (id 2) (at 142.24 54.61 0)
       (effects (font (size 1.27 1.27)) hide)
     )
@@
     (property "License" "BSD-3-Clause" (id 5) (at 142.24 125.73 0)
       (effects (font (size 1.27 1.27)) hide)
+    )
+    (property "Disclaimer" "SEGA and Game Gear are registered trademarks of SEGA GAMES CO., LTD. Not sponsored, endorsed, or approved by SEGA." (id 6) (at 142.24 128.27 0)
+      (effects (font (size 0.5 0.5)) hide)
     )
     (pin "2")
@@
     )
     (path "/1ec0db42-de32-45e9-a7b0-0e03bae3e667"
-      (reference "J1") (unit 1) (value "SG_GG_CARTRIDGE_FINGERS") (footprint "!GGFootprints:SG_GG_CARTRIDGE_FINGERS")
-    )
-  )
+      (reference "J1") (unit 1) (value "SG_GG_CARTRIDGE_FINGERS") (footprint "!SGFootprints:SG_GG_CARTRIDGE_FINGERS")
+    )
+  )
